File: pcb/velopath_final.kicad_sch (KiCad schematic)
At the start: 64 parts, among them J1 charger, J2 battery, J3 control, J4 gnd, J5 ESC_power, J6 control, J7 gnd, P2 SWD, Q6 2SJ168, SW1 Push_Button, U1 LIS3MDL, U3 STM32F103RGTx, Y2 8MHz

Commit message: Sync repository with current project state
Parts:
- removed C26: C,IEC, Capacitor_SMD:C_0603_1608Metric_Pad1.08x0.95mm_HandSolder, symbol PCM_Generic:C,IEC
- removed R8: 110 kOm, PCM_4ms_Resistor:R_0402, symbol PCM_Generic:R,IEC
- added R18: 2k, Resistor_SMD:R_0603_1608Metric_Pad0.98x0.95mm_HandSolder, symbol PCM_Generic:R,IEC
- C18, C19: value 10 uF -> 22 uF
- C23, C24: value C,IEC -> 100nF
- C25: value C,IEC -> 10nF
- D1, D10, D11, D2, JP1: value ~ -> (none)
- J2: footprint PCM_SparkFun-Connector:1x03_P2.54mm -> Connector_PinSocket_2.54mm:PinSocket_1x03_P2.54mm_Vertical
- Q1: value ~ -> HY2122-AB1B
- Q2, Q3: value ~ -> N-MOSFET 30V logic-level; symbol PCM_Generic:Q-BJT,NPN,IEEE -> Transistor_FET:Q_NMOS_GDS
- R10, R9: value R,IEC -> 470R
- R17: footprint PCM_4ms_Resistor:R_0402 -> Resistor_SMD:R_0402_1005Metric_Pad0.72x0.64mm_HandSolder
- U6: value ~ -> (none); symbol moes:WH-BLE106 -> moes:WH-BLE106_1
- U7: renamed from D7; value ~ -> CN3765; symbol velopath:CN3763 -> velopath:CN3765
Connections:
- net +3.3V: now also D3.3 (VOUT), R17.2 (-); no longer D3.2 (VOUT)
- net B+: now also D3.2 (VIN); no longer D3.3 (VIN)
- net GND: now also R18.1 (+); no longer R17.1 (+)
- net chrg_done: now reaches U7.4
- net chrg_done: now also R17.1 (+), U3.14 (PA0); no longer R17.2 (-)
- net at C25.1 (+), Q1.3: now also R18.2 (-)
- net nReload: now reaches U6.1 (nReload)
- net nReload: now also U3.25 (PC5)
- net Link: now reaches U6.11 (Link)
- net Link: now also U3.21 (PA5)
- net nReset: now reaches U6.12 (nReset)
- net nReset: now also U3.20 (PA4)
- net nWake: now reaches U6.2 (nWake)
- net nWake: now also U3.24 (PC4)
- no-connect marks 52 -> 43
Other:
- note added: "SWD"
- moved on the sheet: C1, C10, C11, C2, C23, C24, C25, C3, C4, C7, C8, C9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
